Commit message: moved robot descriptions into a separate package

File: ariac_description/urdf/gantry_macro.xacro (robot description, xacro)
@@ -13,5 +13,5 @@
     initial_positions">
     <!-- ROS2 Control -->
-    <xacro:include filename="$(find ariac_ros2)/robots/gantry_description/urdf/gantry_ros2_control.xacro"/>
+    <xacro:include filename="$(find ariac_description)/urdf/gantry.ros2_control.xacro"/>
     <xacro:gantry_ros2_control
       name="gantry"
@@ -118,10 +118,10 @@
       <visual>
         <geometry>
-          <mesh filename="file://$(find ariac_ros2)/robots/gantry_description/meshes/torso_base.dae" scale="2 2 2"/>
-        </geometry>
-      </visual>
-      <collision>
-        <geometry>
-          <mesh filename="file://$(find ariac_ros2)/robots/gantry_description/meshes/torso_base.dae" scale="2 2 2"/>
+          <mesh filename="file://$(find ariac_description)/meshes/gantry/torso_base.dae" scale="2 2 2"/>
+        </geometry>
+      </visual>
+      <collision>
+        <geometry>
+          <mesh filename="file://$(find ariac_description)/meshes/gantry/torso_base.dae" scale="2 2 2"/>
         </geometry>
       </collision>
@@ -153,10 +153,10 @@
       <visual>
         <geometry>
-          <mesh filename="file://$(find ariac_ros2)/robots/gantry_description/meshes/torso_fixed_normals.dae" scale="2 2 2"/>
-        </geometry>
-      </visual>
-      <collision>
-        <geometry>
-          <mesh filename="file://$(find ariac_ros2)/robots/gantry_description/meshes/torso_fixed_normals.dae" scale="2 2 2"/>
+          <mesh filename="file://$(find ariac_description)/meshes/gantry/torso_fixed_normals.dae" scale="2 2 2"/>
+        </geometry>
+      </visual>
+      <collision>
+        <geometry>
+          <mesh filename="file://$(find ariac_description)/meshes/gantry/torso_fixed_normals.dae" scale="2 2 2"/>
         </geometry>
       </collision>
@@ -195,5 +195,5 @@
         <origin xyz="0 0 0" rpy="0 0 0" />
         <geometry>
-          <mesh filename="file://$(find ariac_ros2)/models/gantry_tray/mesh/gantry_tray.dae" scale="0.5 0.5 1.2"/>
+          <mesh filename="file://$(find ariac_description)/meshes/gantry/gantry_tray.dae" scale="0.5 0.5 1.2"/>
         </geometry>
       </visual>
@@ -201,5 +201,5 @@
         <origin xyz="0 0 0" rpy="0 0 0" />
         <geometry>
-          <mesh filename="file://$(find ariac_ros2)/models/gantry_tray/mesh/gantry_tray.dae" scale="0.5 0.5 1.2"/>
+          <mesh filename="file://$(find ariac_description)/meshes/gantry/gantry_tray.dae" scale="0.5 0.5 1.2"/>
         </geometry>
       </collision>

File: ariac_description/urdf/kitting_robot.urdf.xacro (robot description, xacro)
@@ -1,31 +1,23 @@
 <?xml version="1.0" ?>
-<robot name="gantry" xmlns:xacro="http://ros.org/wiki/xacro">
-  <!-- Include gantry macro -->
-  <xacro:include filename="$(find ariac_ros2)/robots/gantry_description/urdf/gantry_macro.xacro"/>
+<robot name="kitting_robot" xmlns:xacro="http://ros.org/wiki/xacro">
+  <!-- Include linear actuator macro -->
+  <xacro:include filename="$(find ariac_description)/urdf/linear_actuator_macro.xacro"/>
   <!-- Inclue ur robot macro -->
   <xacro:include filename="$(find ur_description)/urdf/ur_macro.xacro"/>
-  <xacro:arg name="initial_positions_file" default="$(find ariac_ros2)/config/gantry_initial_positions.yaml"/>
+  <xacro:arg name="initial_positions_file" default="$(find ariac_description)/config/kitting_robot_initial_positions.yaml"/>
   <xacro:property name="initial_positions_file" default="$(arg initial_positions_file)"/>
   <!-- Create a world link -->
   <link name="world" />
-  <!-- Run gantry macro -->
-  <xacro:gantry
+  <!-- Run linear actuator macro -->
+  <xacro:linear_actuator
     parent="world"
-    long_rail_length="15.0"
-    long_rail_width="0.2"
-    long_rail_offset="-5.0"
-    small_rail_length="15.0"
-    small_rail_width="0.2"
-    rail_height="2.9"
-    rail_thickness="0.1"
-    torso_height="-2.3"
     initial_positions="${load_yaml(initial_positions_file)}"
     >
-  </xacro:gantry>
+  </xacro:linear_actuator>
   <!-- Run ur macro -->
   <xacro:ur_robot
-    name="$gantry_arm"
+    name="kitting_arm"
     prefix=""
-    parent="torso_main"
+    parent="robot_base"
     joint_limits_parameters_file="$(find ur_description)/config/ur10e/joint_limits.yaml"
     kinematics_parameters_file="$(find ur_description)/config/ur10e/default_kinematics.yaml"
@@ -34,14 +26,13 @@
     sim_gazebo="true"
     initial_positions="${load_yaml(initial_positions_file)}">
-    <origin xyz="0.51 0.0 1.3" rpy="0 1.57 0" />
+    <origin xyz="0 0 0.025" rpy="0 0 0" />
   </xacro:ur_robot>
   <gazebo
     reference="world">
   </gazebo>
-  <xacro:arg name="arm_controllers" default="$(find ariac_ros2)/robots/gantry_description/controller/gantry_arm_controllers.yaml" />
-  <!-- <xacro:arg name="gantry_controllers" default="$(find ariac_ros2)/robots/gantry_description/controller/gantry_control.yaml" /> -->
+  <xacro:arg name="controllers" default="$(find ariac_description)/config/kitting_robot_controllers.yaml" />
   <gazebo>
     <plugin filename="libgazebo_ros2_control.so" name="gazebo_ros2_control">
-      <parameters>$(arg arm_controllers)</parameters>
+      <parameters>$(arg controllers)</parameters>
     </plugin>
   </gazebo>
