Commit message: fixed position of kitting robot

File: ariac_description/urdf/linear_actuator_macro.xacro (robot description, xacro)
@@ -34,5 +34,5 @@
       <parent link="${parent}"/>
       <child link="slide_bar"/>
-      <origin xyz="0.0 0.0 0.5" rpy="0.0 0.0 ${-pi/2}"/>
+      <origin xyz="-1.3 0.0 0.9" rpy="0.0 0.0 ${pi}"/>
     </joint>
     <joint name="linear_actuator" type="prismatic">
@@ -41,5 +41,5 @@
       <parent link="slide_bar"/>
       <child link="robot_base"/>
-      <limit effort="1000.0" lower="-4.8" upper="4.8" velocity="5"/>
+      <limit effort="1000.0" lower="-4.8" upper="4.8" velocity="4"/>
       <dynamics damping="20.0" friction="500.0" />
     </joint>
