Commit message: completed refactor of renaming assembly robot to ceiling robot and kitting robot to floor robot

File: ariac_description/urdf/ceiling_robot.urdf.xacro (robot description, xacro)
@@ -1,23 +1,31 @@
 <?xml version="1.0" ?>
-<robot name="kitting_robot" xmlns:xacro="http://ros.org/wiki/xacro">
-  <!-- Include linear actuator macro -->
-  <xacro:include filename="$(find ariac_description)/urdf/linear_actuator_macro.xacro"/>
+<robot name="ceiling_robot" xmlns:xacro="http://ros.org/wiki/xacro">
+  <!-- Include gantry macro -->
+  <xacro:include filename="$(find ariac_description)/urdf/gantry_macro.xacro"/>
   <!-- Inclue ur robot macro -->
   <xacro:include filename="$(find ur_description)/urdf/ur_macro.xacro"/>
-  <xacro:arg name="initial_positions_file" default="$(find ariac_description)/config/kitting_robot_initial_positions.yaml"/>
+  <xacro:arg name="initial_positions_file" default="$(find ariac_description)/config/ceiling_robot_initial_positions.yaml"/>
   <xacro:property name="initial_positions_file" default="$(arg initial_positions_file)"/>
   <!-- Create a world link -->
   <link name="world" />
-  <!-- Run linear actuator macro -->
-  <xacro:linear_actuator
+  <!-- Run gantry macro -->
+  <xacro:gantry
     parent="world"
+    long_rail_length="15.0"
+    long_rail_width="0.2"
+    long_rail_offset="-5.0"
+    small_rail_length="15.0"
+    small_rail_width="0.2"
+    rail_height="2.9"
+    rail_thickness="0.1"
+    torso_height="-2.3"
     initial_positions="${load_yaml(initial_positions_file)}"
     >
-  </xacro:linear_actuator>
+  </xacro:gantry>
   <!-- Run ur macro -->
   <xacro:ur_robot
-    name="kitting_arm"
-    prefix="kitting_"
-    parent="robot_base"
+    name="ceiling_arm"
+    prefix="ceiling_"
+    parent="torso_main"
     joint_limits_parameters_file="$(find ur_description)/config/ur10e/joint_limits.yaml"
     kinematics_parameters_file="$(find ur_description)/config/ur10e/default_kinematics.yaml"
@@ -26,17 +34,17 @@
     sim_gazebo="true"
     initial_positions="${load_yaml(initial_positions_file)}">
-    <origin xyz="0 0 0.025" rpy="0 0 0" />
+    <origin xyz="0.51 0.0 1.3" rpy="0 1.57 0" />
   </xacro:ur_robot>
   <gazebo
     reference="world">
   </gazebo>
-  <xacro:arg name="controllers" default="$(find ariac_description)/config/kitting_robot_controllers.yaml" />
+  <xacro:arg name="controllers" default="$(find ariac_description)/config/ceiling_robot_controllers.yaml" />
   <gazebo>
     <plugin filename="libgazebo_ros2_control.so" name="gazebo_ros2_control">
       <ros>
-        <namespace>/kitting</namespace>
+        <namespace>/ceiling</namespace>
       </ros>
       <parameters>$(arg controllers)</parameters>
-      <robot_param_node>/kitting/robot_state_publisher</robot_param_node>
+      <robot_param_node>/ceiling/robot_state_publisher</robot_param_node>
     </plugin>
   </gazebo>

File: ariac_description/urdf/floor_robot.urdf.xacro (robot description, xacro)
@@ -1,31 +1,23 @@
 <?xml version="1.0" ?>
-<robot name="assembly_robot" xmlns:xacro="http://ros.org/wiki/xacro">
-  <!-- Include gantry macro -->
-  <xacro:include filename="$(find ariac_description)/urdf/gantry_macro.xacro"/>
+<robot name="floor_robot" xmlns:xacro="http://ros.org/wiki/xacro">
+  <!-- Include linear actuator macro -->
+  <xacro:include filename="$(find ariac_description)/urdf/linear_actuator_macro.xacro"/>
   <!-- Inclue ur robot macro -->
   <xacro:include filename="$(find ur_description)/urdf/ur_macro.xacro"/>
-  <xacro:arg name="initial_positions_file" default="$(find ariac_description)/config/assembly_robot_initial_positions.yaml"/>
+  <xacro:arg name="initial_positions_file" default="$(find ariac_description)/config/floor_robot_initial_positions.yaml"/>
   <xacro:property name="initial_positions_file" default="$(arg initial_positions_file)"/>
   <!-- Create a world link -->
   <link name="world" />
-  <!-- Run gantry macro -->
-  <xacro:gantry
+  <!-- Run linear actuator macro -->
+  <xacro:linear_actuator
     parent="world"
-    long_rail_length="15.0"
-    long_rail_width="0.2"
-    long_rail_offset="-5.0"
-    small_rail_length="15.0"
-    small_rail_width="0.2"
-    rail_height="2.9"
-    rail_thickness="0.1"
-    torso_height="-2.3"
     initial_positions="${load_yaml(initial_positions_file)}"
     >
-  </xacro:gantry>
+  </xacro:linear_actuator>
   <!-- Run ur macro -->
   <xacro:ur_robot
-    name="assembly_arm"
-    prefix="assembly_"
-    parent="torso_main"
+    name="floor_arm"
+    prefix="floor_"
+    parent="robot_base"
     joint_limits_parameters_file="$(find ur_description)/config/ur10e/joint_limits.yaml"
     kinematics_parameters_file="$(find ur_description)/config/ur10e/default_kinematics.yaml"
@@ -34,17 +26,17 @@
     sim_gazebo="true"
     initial_positions="${load_yaml(initial_positions_file)}">
-    <origin xyz="0.51 0.0 1.3" rpy="0 1.57 0" />
+    <origin xyz="0 0 0.025" rpy="0 0 0" />
   </xacro:ur_robot>
   <gazebo
     reference="world">
   </gazebo>
-  <xacro:arg name="controllers" default="$(find ariac_description)/config/assembly_robot_controllers.yaml" />
+  <xacro:arg name="controllers" default="$(find ariac_description)/config/floor_robot_controllers.yaml" />
   <gazebo>
     <plugin filename="libgazebo_ros2_control.so" name="gazebo_ros2_control">
       <ros>
-        <namespace>/assembly</namespace>
+        <namespace>/floor</namespace>
       </ros>
       <parameters>$(arg controllers)</parameters>
-      <robot_param_node>/assembly/robot_state_publisher</robot_param_node>
+      <robot_param_node>/floor/robot_state_publisher</robot_param_node>
     </plugin>
   </gazebo>
