Commit message: updated agv_bringup to start all four agvs

File: ariac_description/urdf/AGV/agv.urdf.xacro (robot description, xacro)
@@ -3,9 +3,14 @@
   <!-- Include macro -->
   <xacro:include filename="$(find ariac_description)/urdf/AGV/agv_macro.xacro"/>
+  <xacro:arg name="agv_number" default="agv_1"/>
+  <xacro:property name="agv_number" default="$(arg agv_number)"/>
+  <xacro:arg name="y_position" default="0"/>
+  <xacro:property name="y_position" default="$(arg y_position)"/>
   <!-- Create a world link -->
   <link name="world"/>
   <!-- Run agv macro -->
   <xacro:agv
-    number="1"
+    agv_number="$(arg agv_number)"
+    y_position="$(arg y_position)"
     >
   </xacro:agv>
@@ -17,8 +22,8 @@
     <plugin filename="libgazebo_ros2_control.so" name="gazebo_ros2_control">
       <ros>
-        <namespace>/agv</namespace>
+        <namespace>/$(arg agv_number)</namespace>
       </ros>
       <parameters>$(arg controllers)</parameters>
-      <robot_param_node>/agv/robot_state_publisher</robot_param_node>
+      <robot_param_node>/$(arg agv_number)/robot_state_publisher</robot_param_node>
     </plugin>
   </gazebo>

File: ariac_description/urdf/AGV/agv_macro.xacro (robot description, xacro)
@@ -2,9 +2,10 @@
 <robot xmlns:xacro="http://wiki.ros.org/xacro">
   <xacro:macro name="agv" params="
-    number">
+    agv_number
+    y_position">
     <xacro:include filename="$(find ariac_description)/urdf/AGV/agv.ros2_control.xacro"/>
     <!-- Run ROS2 control macro -->
     <xacro:agv_ros2_control
-      name="agv"
+      name="$(arg agv_number)"
     />
     <link name="track">
@@ -37,5 +38,5 @@
       <parent link="world"/>
       <child link="track"/>
-      <origin xyz="-2 4.707484 0.0" rpy="0.0 0.0 ${pi/2}"/>
+      <origin xyz="-2 $(arg y_position) 0.0" rpy="0.0 0.0 ${pi/2}"/>
     </joint>
     <joint name="agv_joint" type="prismatic">

File: ariac_description/urdf/gantry_macro.xacro (robot description, xacro)
@@ -108,8 +108,8 @@
       <parent link="long_rail_2"/>
       <child link="small_rail"/>
-      <origin xyz="0.0 0.0 ${rail_height + rail_thickness}" rpy="0.0 0.0 ${pi/2}"/>
+      <origin xyz="0.0 -5.0 ${rail_height + rail_thickness}" rpy="0.0 0.0 ${pi/2}"/>
       <axis xyz="1 0 0"/>
-      <limit lower="${-long_rail_length / 2 + long_rail_offset + small_rail_width / 2}"
-          upper="${long_rail_length / 2 + long_rail_offset - small_rail_width / 2}"
+      <limit lower="${-long_rail_length / 2 + small_rail_width / 2}"
+          upper="${long_rail_length / 2 - small_rail_width / 2}"
           velocity="1"
           effort="100000"/>
