Commit message: added service to move agvs between various stations, added bins, assembly stations and conveyor to world file

File: ariac_description/urdf/AGV/agv_macro.xacro (robot description, xacro)
@@ -56,5 +56,5 @@
       <parent link="world"/>
       <child link="$(arg agv_number)_track"/>
-      <origin xyz="-2 $(arg y_position) 0.0" rpy="0.0 0.0 ${pi/2}"/>
+      <origin xyz="-2.27 $(arg y_position) 0.0" rpy="0.0 0.0 ${pi/2}"/>
     </joint>
     <joint name="agv_joint" type="prismatic">
@@ -63,5 +63,5 @@
       <parent link="$(arg agv_number)_track"/>
       <child link="$(arg agv_number)_base"/>
-      <limit effort="1000.0" lower="0" upper="12" velocity="10"/>
+      <limit effort="1000.0" lower="0" upper="11" velocity="10"/>
       <dynamics damping="20.0" friction="500.0" />
     </joint>

File: ariac_description/urdf/linear_actuator_macro.xacro (robot description, xacro)
@@ -13,11 +13,13 @@
       <visual>
         <geometry>
-          <box size="0.05 10 0.05"/>
+          <box size="0.2 10 0.1"/>
         </geometry>
         <origin xyz="0 0 0"/>
-        <material name="green">
-          <color rgba="0 0.8 .8 1"/>
-        </material>
       </visual>
+      <collision>
+        <geometry>
+          <box size="0.2 10 0.1"/>
+        </geometry>
+      </collision>
       <inertial>
         <mass value="100"/>
@@ -31,8 +33,11 @@
       </inertial>
     </link>
+    <gazebo reference="slide_bar">
+      <material>Gazebo/Gray</material>
+    </gazebo>
     <joint name="world_to_base" type="fixed">
       <parent link="${parent}"/>
       <child link="slide_bar"/>
-      <origin xyz="-1.3 0.0 0.9" rpy="0.0 0.0 ${pi}"/>
+      <origin xyz="-1.3 0.0 0.93" rpy="0.0 0.0 ${pi}"/>
     </joint>
     <joint name="linear_actuator" type="prismatic">

Commit message: minor updates

File: ariac_description/urdf/AGV/agv_macro.xacro (robot description, xacro)
@@ -6,6 +6,6 @@
     <xacro:include filename="$(find ariac_description)/urdf/AGV/agv.ros2_control.xacro"/>
     <!-- Run ROS2 control macro -->
-    <xacro:agv_ros2_control name="$(arg agv_number)"/>
-    <link name="$(arg agv_number)_track">
+    <xacro:agv_ros2_control name="${agv_number}"/>
+    <link name="${agv_number}_track">
       <inertial>
         <mass value="100"/>
@@ -13,5 +13,5 @@
       </inertial>
     </link>
-    <link name="$(arg agv_number)_base">
+    <link name="${agv_number}_base">
       <visual>
         <geometry>
@@ -33,5 +33,5 @@
       </inertial>
     </link>
-    <link name="$(arg agv_number)_tray">
+    <link name="${agv_number}_tray">
       <visual>
         <geometry>
@@ -50,23 +50,23 @@
       </inertial>
     </link>
-    <gazebo reference="$(arg agv_number)_tray">
+    <gazebo reference="${agv_number}_tray">
       <material>Gazebo/Gray</material>
     </gazebo>
     <joint name="world_to_track" type="fixed">
       <parent link="world"/>
-      <child link="$(arg agv_number)_track"/>
-      <origin xyz="-2.27 $(arg y_position) 0.0" rpy="0.0 0.0 ${pi/2}"/>
+      <child link="${agv_number}_track"/>
+      <origin xyz="-2.27 ${y_position} 0.0" rpy="0.0 0.0 ${pi/2}"/>
     </joint>
     <joint name="agv_joint" type="prismatic">
       <axis xyz="0 1 0"/>
       <origin xyz="0.0 0.0 0.0"/>
-      <parent link="$(arg agv_number)_track"/>
-      <child link="$(arg agv_number)_base"/>
+      <parent link="${agv_number}_track"/>
+      <child link="${agv_number}_base"/>
       <limit effort="1000.0" lower="0" upper="11" velocity="10"/>
       <dynamics damping="20.0" friction="500.0" />
     </joint>
     <joint name="kit_tray" type="fixed">
-      <parent link="$(arg agv_number)_base"/>
-      <child link="$(arg agv_number)_tray"/>
+      <parent link="${agv_number}_base"/>
+      <child link="${agv_number}_tray"/>
       <origin xyz="0 -0.2 0.75" rpy="0.0 0.0 0.0"/>
     </joint>

Commit message: added move agv services for each agv

File: ariac_description/urdf/AGV/agv_macro.xacro (robot description, xacro)
@@ -4,4 +4,7 @@
     agv_number
     y_position">
+    <material name="Grey">
+      <color rgba="${220/255} ${220/255} ${220/255} 1.0"/>
+    </material>
     <xacro:include filename="$(find ariac_description)/urdf/AGV/agv.ros2_control.xacro"/>
     <!-- Run ROS2 control macro -->
@@ -38,4 +41,5 @@
           <mesh filename="file://$(find ariac_description)/meshes/AGV/kit_tray.stl" scale="1 1 1"/>
         </geometry>
+        <material name="Grey"/>
       </visual>
       <collision>

File: ariac_description/urdf/vacuum_gripper/vacuum_gripper_macro.xacro (robot description, xacro)
@@ -55,4 +55,5 @@
         </ros>
         <gripper_link>${prefix}_gripper</gripper_link>
+        <robot_name>${prefix}_robot</robot_name>
       </plugin>
     </gazebo>

Commit message: updated environment to match sketchup file

File: ariac_description/urdf/AGV/agv_macro.xacro (robot description, xacro)
@@ -60,5 +60,5 @@
       <parent link="world"/>
       <child link="${agv_number}_track"/>
-      <origin xyz="-2.27 ${y_position} 0.0" rpy="0.0 0.0 ${pi/2}"/>
+      <origin xyz="-2.27 ${y_position} 0.01" rpy="0.0 0.0 ${pi/2}"/>
     </joint>
     <joint name="${agv_number}_joint" type="prismatic">

Commit message: updated agvs to be able to move to warehouse

File: ariac_description/urdf/AGV/agv_macro.xacro (robot description, xacro)
@@ -67,5 +67,5 @@
       <parent link="${agv_number}_track"/>
       <child link="${agv_number}_base"/>
-      <limit effort="1000.0" lower="0" upper="11" velocity="10"/>
+      <limit effort="1000.0" lower="0" upper="18" velocity="8"/>
       <dynamics damping="20.0" friction="500.0" />
     </joint>

Commit message: added part and tray spawning on AGVS

File: ariac_description/urdf/AGV/agv_macro.xacro (robot description, xacro)
@@ -70,7 +70,9 @@
       <dynamics damping="20.0" friction="500.0" />
     </joint>
-    <joint name="${agv_number}_kit_tray_joint" type="fixed">
+    <joint name="${agv_number}_kit_tray_joint" type="revolute">
+      <axis xyz="0 0 1"/>
       <parent link="${agv_number}_base"/>
       <child link="${agv_number}_tray"/>
+      <limit lower="-.001" upper=".001" effort="0" velocity="0" />
       <origin xyz="0 -0.2 0.75" rpy="0.0 0.0 0.0"/>
     </joint>

Commit message: added plugin to with service to lock and unlock the kit tray to the agv

File: ariac_description/urdf/AGV/agv_macro.xacro (robot description, xacro)
@@ -39,11 +39,16 @@
       <visual>
         <geometry>
-          <mesh filename="file://$(find ariac_description)/meshes/AGV/kit_tray.stl" scale="1 1 1"/>
+          <mesh filename="file://$(find ariac_description)/meshes/AGV/tray.stl" scale="1 1 1"/>
         </geometry>
         <material name="Grey"/>
       </visual>
-      <collision>
+      <collision name="${agv_number}_tray_collision">
         <geometry>
-          <mesh filename="file://$(find ariac_description)/meshes/AGV/kit_tray.stl" scale="1 1 1"/>
+          <mesh filename="file://$(find ariac_description)/meshes/AGV/tray.stl" scale="1 1 1"/>
+        </geometry>
+      </collision>
+      <collision name="${agv_number}_tray_collision1">
+        <geometry>
+          <mesh filename="file://$(find ariac_description)/meshes/AGV/contact_sensor.stl" scale="1 1 1"/>
         </geometry>
       </collision>
@@ -54,4 +59,21 @@
       </inertial>
     </link>
+    <gazebo reference="${agv_number}_tray">
+      <sensor type="contact" name="bumper">
+        <update_rate>10</update_rate>
+        <contact>
+          <collision>${agv_number}_tray_collision1_collision_1</collision>
+        </contact>
+      </sensor>
+    </gazebo>
+    <gazebo>
+      <plugin filename="libAGVTrayPlugin.so" name="${agv_number}_tray_plugin">
+        <ros>
+          <namespace></namespace>
+        </ros>
+        <agv_tray_link>${agv_number}_tray</agv_tray_link>
+        <agv_number>${agv_number}</agv_number>
+      </plugin>
+    </gazebo>
     <gazebo reference="${agv_number}_tray">
       <material>Gazebo/Gray</material>
@@ -70,10 +92,10 @@
       <dynamics damping="20.0" friction="500.0" />
     </joint>
-    <joint name="${agv_number}_kit_tray_joint" type="revolute">
+    <joint name="${agv_number}_tray_joint" type="revolute">
       <axis xyz="0 0 1"/>
       <parent link="${agv_number}_base"/>
       <child link="${agv_number}_tray"/>
       <limit lower="-.001" upper=".001" effort="0" velocity="0" />
-      <origin xyz="0 -0.2 0.75" rpy="0.0 0.0 0.0"/>
+      <origin xyz="0 -0.2 .75" rpy="0.0 0.0 0.0"/>
     </joint>
   </xacro:macro>
