Commit message: added the kit tray to the agv urdf

File: ariac_description/urdf/AGV/agv.ros2_control.xacro (robot description, xacro)
@@ -1,6 +1,5 @@
 <?xml version="1.0"?>
 <robot xmlns:xacro="http://www.ros.org/wiki/xacro">
-  <xacro:macro name="agv_ros2_control" params="
-    name">
+  <xacro:macro name="agv_ros2_control" params="name">
     <ros2_control name="${name}" type="system">
       <hardware>
@@ -8,14 +7,14 @@
       </hardware>
       <joint name="agv_joint">
-      <command_interface name="position">
-        <param name="min">0</param>
-        <param name="max">5</param>
-      </command_interface>
-      <state_interface name="position">
-        <param name="initial_value">0</param>
-      </state_interface>
-      <state_interface name="velocity"/>
-      <state_interface name="effort"/>
-    </joint>
+        <command_interface name="position">
+          <param name="min">0</param>
+          <param name="max">5</param>
+        </command_interface>
+        <state_interface name="position">
+          <param name="initial_value">0</param>
+        </state_interface>
+        <state_interface name="velocity"/>
+        <state_interface name="effort"/>
+      </joint>
     </ros2_control>
   </xacro:macro>

File: ariac_description/urdf/AGV/agv_macro.xacro (robot description, xacro)
@@ -6,8 +6,6 @@
     <xacro:include filename="$(find ariac_description)/urdf/AGV/agv.ros2_control.xacro"/>
     <!-- Run ROS2 control macro -->
-    <xacro:agv_ros2_control
-      name="$(arg agv_number)"
-    />
-    <link name="track">
+    <xacro:agv_ros2_control name="$(arg agv_number)"/>
+    <link name="$(arg agv_number)_track">
       <inertial>
         <mass value="100"/>
@@ -15,5 +13,5 @@
       </inertial>
     </link>
-    <link name="agv">
+    <link name="$(arg agv_number)_base">
       <visual>
         <geometry>
@@ -35,7 +33,27 @@
       </inertial>
     </link>
+    <link name="$(arg agv_number)_tray">
+      <visual>
+        <geometry>
+          <mesh filename="file://$(find ariac_description)/meshes/AGV/kit_tray.stl" scale="1 1 1"/>
+        </geometry>
+      </visual>
+      <collision>
+        <geometry>
+          <mesh filename="file://$(find ariac_description)/meshes/AGV/kit_tray.stl" scale="1 1 1"/>
+        </geometry>
+      </collision>
+      <inertial>
+        <origin xyz="0 0 0" rpy="0 0 0"/>
+        <mass value="1"/>
+        <inertia ixx="0.0408" ixy="0.0" ixz="0.0" iyy="0.02084" iyz="0.0" izz="0.0616"/>
+      </inertial>
+    </link>
+    <gazebo reference="$(arg agv_number)_tray">
+      <material>Gazebo/Gray</material>
+    </gazebo>
     <joint name="world_to_track" type="fixed">
       <parent link="world"/>
-      <child link="track"/>
+      <child link="$(arg agv_number)_track"/>
       <origin xyz="-2 $(arg y_position) 0.0" rpy="0.0 0.0 ${pi/2}"/>
     </joint>
@@ -43,9 +61,14 @@
       <axis xyz="0 1 0"/>
       <origin xyz="0.0 0.0 0.0"/>
-      <parent link="track"/>
-      <child link="agv"/>
+      <parent link="$(arg agv_number)_track"/>
+      <child link="$(arg agv_number)_base"/>
       <limit effort="1000.0" lower="0" upper="12" velocity="10"/>
       <dynamics damping="20.0" friction="500.0" />
     </joint>
+    <joint name="kit_tray" type="fixed">
+      <parent link="$(arg agv_number)_base"/>
+      <child link="$(arg agv_number)_tray"/>
+      <origin xyz="0 -0.2 0.75" rpy="0.0 0.0 0.0"/>
+    </joint>
   </xacro:macro>
 </robot>

Commit message: changes to launch configuration of robots

File: ariac_description/urdf/AGV/agv.ros2_control.xacro (robot description, xacro)
@@ -2,22 +2,17 @@
 <robot xmlns:xacro="http://www.ros.org/wiki/xacro">
   <xacro:macro name="agv_ros2_control" params="name">
-    <ros2_control name="${name}" type="system">
+    <ros2_control name="${name}_ros2_control" type="system">
       <hardware>
         <plugin>gazebo_ros2_control/GazeboSystem</plugin>
       </hardware>
-      <joint name="agv_joint">
+      <joint name="${name}_joint">
         <command_interface name="velocity">
           <param name="min">0</param>
           <param name="max">5</param>
         </command_interface>
-        <!-- <command_interface name="effort">
-          <param name="min">0</param>
-          <param name="max">5</param>
-        </command_interface> -->
         <state_interface name="position">
           <param name="initial_value">0</param>
         </state_interface>
         <state_interface name="velocity"/>
-        <!-- <state_interface name="effort"/> -->
       </joint>
     </ros2_control>

File: ariac_description/urdf/AGV/agv.urdf.xacro (robot description, xacro)
@@ -18,9 +18,9 @@
     reference="world">
   </gazebo>
-  <xacro:arg name="controllers" default="$(find ariac_description)/config/agv_controllers.yaml" />
+  <xacro:arg name="controllers" default="$(find ariac_description)/config/$(arg agv_number)_controllers.yaml" />
   <gazebo>
     <plugin filename="libgazebo_ros2_control.so" name="$(arg agv_number)_gazebo_ros2_control">
       <ros>
-        <namespace>/$(arg agv_number)</namespace>
+        <namespace>$(arg agv_number)</namespace>
       </ros>
       <parameters>$(arg controllers)</parameters>
@@ -28,3 +28,12 @@
     </plugin>
   </gazebo>
+  <!-- Create ARIAC AGV plugin -->
+  <gazebo>
+    <plugin filename="libagv_plugin.so" name="$(arg agv_number)_plugin">
+      <ros>
+        <namespace>$(arg agv_number)</namespace>
+      </ros>
+      <agv_number>$(arg agv_number)</agv_number>
+    </plugin>
+  </gazebo>
 </robot>

File: ariac_description/urdf/AGV/agv_macro.xacro (robot description, xacro)
@@ -53,10 +53,10 @@
       <material>Gazebo/Gray</material>
     </gazebo>
-    <joint name="world_to_track" type="fixed">
+    <joint name="${agv_number}_world_to_track" type="fixed">
       <parent link="world"/>
       <child link="${agv_number}_track"/>
       <origin xyz="-2.27 ${y_position} 0.0" rpy="0.0 0.0 ${pi/2}"/>
     </joint>
-    <joint name="agv_joint" type="prismatic">
+    <joint name="${agv_number}_joint" type="prismatic">
       <axis xyz="0 1 0"/>
       <origin xyz="0.0 0.0 0.0"/>
@@ -66,5 +66,5 @@
       <dynamics damping="20.0" friction="500.0" />
     </joint>
-    <joint name="kit_tray" type="fixed">
+    <joint name="${agv_number}_kit_tray_joint" type="fixed">
       <parent link="${agv_number}_base"/>
       <child link="${agv_number}_tray"/>

Commit message: updates to put robot state publisher back into a namespace

File: ariac_description/urdf/AGV/agv.ros2_control.xacro (robot description, xacro)
@@ -16,4 +16,9 @@
         <state_interface name="velocity"/>
       </joint>
+      <joint name="${name}_kit_tray_joint">
+        <state_interface name="position">
+          <param name="initial_value">0</param>
+        </state_interface>
+      </joint>
     </ros2_control>
   </xacro:macro>

File: ariac_description/urdf/AGV/agv.urdf.xacro (robot description, xacro)
@@ -24,5 +24,5 @@
       </ros>
       <parameters>$(arg controllers)</parameters>
-      <robot_param_node>/$(arg agv_number)_robot_state_publisher</robot_param_node>
+      <robot_param_node>/$(arg agv_number)/robot_state_publisher</robot_param_node>
       <controller_manager_prefix>$(arg agv_number)</controller_manager_prefix>
     </plugin>

File: ariac_description/urdf/ceiling_robot/ceiling_robot.urdf.xacro (robot description, xacro)
@@ -53,5 +53,5 @@
       </ros>
       <parameters>$(arg controllers)</parameters>
-      <robot_param_node>/ceiling_robot_robot_state_publisher</robot_param_node>
+      <robot_param_node>/ceiling_robot/robot_state_publisher</robot_param_node>
       <controller_manager_prefix>ceiling_robot</controller_manager_prefix>
     </plugin>

File: ariac_description/urdf/floor_robot/floor_robot.urdf.xacro (robot description, xacro)
@@ -45,5 +45,5 @@
       </ros>
       <parameters>$(arg controllers)</parameters>
-      <robot_param_node>/floor_robot_robot_state_publisher</robot_param_node>
+      <robot_param_node>/floor_robot/robot_state_publisher</robot_param_node>
       <controller_manager_prefix>floor_robot</controller_manager_prefix>
     </plugin>

Commit message: Revert "Navigation"

File: ariac_description/urdf/AGV/agv.ros2_control.xacro (robot description, xacro)
@@ -2,10 +2,10 @@
 <robot xmlns:xacro="http://www.ros.org/wiki/xacro">
   <xacro:macro name="agv_ros2_control" params="name">
-    <ros2_control name="${name}_ros2_control" type="system">
+    <ros2_control name="${name}" type="system">
       <hardware>
         <plugin>gazebo_ros2_control/GazeboSystem</plugin>
       </hardware>
-      <joint name="${name}_joint">
-        <command_interface name="velocity">
+      <joint name="agv_joint">
+        <command_interface name="position">
           <param name="min">0</param>
           <param name="max">5</param>
@@ -15,4 +15,5 @@
         </state_interface>
         <state_interface name="velocity"/>
+        <state_interface name="effort"/>
       </joint>
     </ros2_control>

File: ariac_description/urdf/AGV/agv.urdf.xacro (robot description, xacro)
@@ -18,9 +18,9 @@
     reference="world">
   </gazebo>
-  <xacro:arg name="controllers" default="$(find ariac_description)/config/$(arg agv_number)_controllers.yaml" />
+  <xacro:arg name="controllers" default="$(find ariac_description)/config/agv_controllers.yaml" />
   <gazebo>
     <plugin filename="libgazebo_ros2_control.so" name="$(arg agv_number)_gazebo_ros2_control">
       <ros>
-        <namespace>$(arg agv_number)</namespace>
+        <namespace>/$(arg agv_number)</namespace>
       </ros>
       <parameters>$(arg controllers)</parameters>
@@ -28,12 +28,3 @@
     </plugin>
   </gazebo>
-  <!-- Create ARIAC AGV plugin -->
-  <gazebo>
-    <plugin filename="libagv_plugin.so" name="$(arg agv_number)_plugin">
-      <ros>
-        <namespace>$(arg agv_number)</namespace>
-      </ros>
-      <agv_number>$(arg agv_number)</agv_number>
-    </plugin>
-  </gazebo>
 </robot>

File: ariac_description/urdf/AGV/agv_macro.xacro (robot description, xacro)
@@ -4,7 +4,4 @@
     agv_number
     y_position">
-    <material name="Grey">
-      <color rgba="${220/255} ${220/255} ${220/255} 1.0"/>
-    </material>
     <xacro:include filename="$(find ariac_description)/urdf/AGV/agv.ros2_control.xacro"/>
     <!-- Run ROS2 control macro -->
@@ -41,5 +38,4 @@
           <mesh filename="file://$(find ariac_description)/meshes/AGV/kit_tray.stl" scale="1 1 1"/>
         </geometry>
-        <material name="Grey"/>
       </visual>
       <collision>
@@ -57,18 +53,18 @@
       <material>Gazebo/Gray</material>
     </gazebo>
-    <joint name="${agv_number}_world_to_track" type="fixed">
+    <joint name="world_to_track" type="fixed">
       <parent link="world"/>
       <child link="${agv_number}_track"/>
-      <origin xyz="-2.27 ${y_position} 0.01" rpy="0.0 0.0 ${pi/2}"/>
+      <origin xyz="-2.27 ${y_position} 0.0" rpy="0.0 0.0 ${pi/2}"/>
     </joint>
-    <joint name="${agv_number}_joint" type="prismatic">
+    <joint name="agv_joint" type="prismatic">
       <axis xyz="0 1 0"/>
       <origin xyz="0.0 0.0 0.0"/>
       <parent link="${agv_number}_track"/>
       <child link="${agv_number}_base"/>
-      <limit effort="1000.0" lower="0" upper="18" velocity="8"/>
+      <limit effort="1000.0" lower="0" upper="11" velocity="10"/>
       <dynamics damping="20.0" friction="500.0" />
     </joint>
-    <joint name="${agv_number}_kit_tray_joint" type="fixed">
+    <joint name="kit_tray" type="fixed">
       <parent link="${agv_number}_base"/>
       <child link="${agv_number}_tray"/>

File: ariac_description/urdf/floor_robot/floor_robot.urdf.xacro (robot description, xacro)
@@ -28,5 +28,5 @@
     sim_gazebo="true"
     initial_positions="${load_yaml(initial_positions_file)}">
-    <origin xyz="0 0 0.05" rpy="0 0 0" />
+    <origin xyz="0 0 0.025" rpy="0 0 0" />
   </xacro:ur_robot>
   <!-- Run gripper macro -->

File: ariac_description/urdf/vacuum_gripper/vacuum_gripper_macro.xacro (robot description, xacro)
@@ -5,15 +5,12 @@
     prefix">
     <link name="${prefix}_gripper">
-      <visual name="${prefix}_gripper_visual">
-        <origin xyz="0 0 0" rpy="0 0 0"/>
+      <visual>
         <geometry>
           <mesh filename="file://$(find ariac_description)/meshes/vacuum_gripper/vacuum_gripper.stl" scale="1 1 1"/>
         </geometry>
       </visual>
-      <collision name="${prefix}_gripper_collision">
-        <origin xyz="0 0 -0.005" rpy="0 0 0"/>
+      <collision>
         <geometry>
-          <!-- <mesh filename="file://$(find ariac_description)/meshes/vacuum_gripper/vacuum_gripper.stl" scale="1 1 1"/> -->
-          <cylinder radius="0.05" length="0.01" />
+          <mesh filename="file://$(find ariac_description)/meshes/vacuum_gripper/vacuum_gripper.stl" scale="1 1 1"/>
         </geometry>
       </collision>
@@ -25,54 +22,23 @@
     </link>
     <gazebo reference="${prefix}_gripper">
-      <visual name="${prefix}_gripper_visual">
-        <origin xyz="0 0 0" rpy="0 0 0"/>
-        <geometry>
-          <!-- <mesh filename="file://$(find ariac_description)/meshes/vacuum_gripper/vacuum_gripper.stl" scale="1 1 1"/> -->
-        </geometry>
-        <plugin filename="libgripper_change_plugin.so" name="${prefix}_gripper_change_plugin">
-          <ros>
-          </ros>
-          <robot_name>${prefix}_robot</robot_name>
-        </plugin>
-      </visual>
-    </gazebo>
-    <gazebo reference="${prefix}_gripper">
       <material>Gazebo/Black</material>
     </gazebo>
-    <joint name="${prefix}_gripper_joint" type="revolute">
-      <axis xyz="0 0 1"/>
+    <joint name="${prefix}_robot_to_gripper" type="fixed">
       <parent link="${prefix}_${parent}"/>
       <child link="${prefix}_gripper"/>
-      <limit lower="-.1" upper=".1" effort="0" velocity="0" />
       <origin xyz="0.0 0.0 0.01" rpy="0.0 0.0 0.0"/>
     </joint>
-    <!-- Add a contact sensor to the gripper -->
-    <gazebo reference="${prefix}_gripper">
-      <sensor type="contact" name="bumper">
-        <update_rate>10</update_rate>
-        <contact>
-          <collision>${prefix}_gripper_collision_collision</collision>
-        </contact>
-      </sensor>
-    </gazebo>
-    <gazebo>
-      <plugin filename="libvacuum_gripper.so" name="${prefix}_vacuum_gripper_plugin">
+    <!-- <gazebo>
+      <plugin name='vacuum_gripper' filename='libgazebo_ros_vacuum_gripper.so'>
         <ros>
-          <namespace>${prefix}_robot</namespace>
+          <namespace>/${prefix}</namespace>
+          <remapping>switch:=activate_gripper</remapping>
+          <remapping>grasping:=gripper_state</remapping>
         </ros>
-        <gripper_link>${prefix}_gripper</gripper_link>
-        <robot_name>${prefix}_robot</robot_name>
+        <link_name>${prefix}_gripper</link_name>
+        <max_distance>10.0</max_distance>
+        <fixed>ground_plane</fixed>
       </plugin>
-    </gazebo>
-    <ros2_control name="${prefix}_gripper_control" type="system">
-      <hardware>
-        <plugin>gazebo_ros2_control/GazeboSystem</plugin>
-      </hardware>
-      <joint name="${prefix}_gripper_joint">
-        <state_interface name="position">
-          <param name="initial_value">0</param>
-        </state_interface>
-      </joint>
-    </ros2_control>
+    </gazebo> -->
   </xacro:macro>
 </robot>

Commit message: fixed issues with moveit

File: ariac_description/urdf/AGV/agv.ros2_control.xacro (robot description, xacro)
@@ -16,5 +16,5 @@
         <state_interface name="velocity"/>
       </joint>
-      <joint name="${name}_kit_tray_joint">
+      <joint name="${name}_tray_joint">
         <state_interface name="position">
           <param name="initial_value">0</param>

File: ariac_description/urdf/AGV/agv.urdf.xacro (robot description, xacro)
@@ -22,4 +22,5 @@
     <plugin filename="libgazebo_ros2_control.so" name="$(arg agv_number)_gazebo_ros2_control">
       <ros>
+        <namespace>$(arg agv_number)</namespace>
       </ros>
       <parameters>$(arg controllers)</parameters>

File: ariac_description/urdf/ceiling_robot/ceiling_robot.urdf.xacro (robot description, xacro)
@@ -51,4 +51,5 @@
     <plugin filename="libgazebo_ros2_control.so" name="ceiling_robot_gazebo_ros2_control">
       <ros>
+        <namespace>ceiling_robot</namespace>
       </ros>
       <parameters>$(arg controllers)</parameters>

File: ariac_description/urdf/floor_robot/floor_robot.urdf.xacro (robot description, xacro)
@@ -43,4 +43,5 @@
     <plugin filename="libgazebo_ros2_control.so" name="floor_robot_gazebo_ros2_control">
       <ros>
+        <namespace>floor_robot</namespace>
       </ros>
       <parameters>$(arg controllers)</parameters>

File: ariac_description/urdf/vacuum_gripper/vacuum_gripper_macro.xacro (robot description, xacro)
@@ -24,9 +24,8 @@
       </inertial>
     </link>
-    <gazebo reference="${prefix}_gripper">
+    <!-- <gazebo reference="${prefix}_gripper">
       <visual name="${prefix}_gripper_visual">
         <origin xyz="0 0 0" rpy="0 0 0"/>
         <geometry>
-          <!-- <mesh filename="file://$(find ariac_description)/meshes/vacuum_gripper/vacuum_gripper.stl" scale="1 1 1"/> -->
         </geometry>
         <plugin filename="libgripper_change_plugin.so" name="${prefix}_gripper_change_plugin">
@@ -36,5 +35,5 @@
         </plugin>
       </visual>
-    </gazebo>
+    </gazebo> -->
     <gazebo reference="${prefix}_gripper">
       <material>Gazebo/Black</material>
