Commit message: cleaned up description package

File: ariac_description/urdf/ceiling_robot/ceiling_robot.urdf.xacro (robot description, xacro)
@@ -1,25 +1,33 @@
 <?xml version="1.0" ?>
-<robot name="floor_robot" xmlns:xacro="http://ros.org/wiki/xacro">
-  <!-- Include linear actuator macro -->
-  <xacro:include filename="$(find ariac_description)/urdf/linear_actuator_macro.xacro"/>
+<robot name="ceiling_robot" xmlns:xacro="http://ros.org/wiki/xacro">
+  <!-- Include gantry macro -->
+  <xacro:include filename="$(find ariac_description)/urdf/ceiling_robot/gantry_macro.xacro"/>
   <!-- Inclue ur robot macro -->
   <xacro:include filename="$(find ur_description)/urdf/ur_macro.xacro"/>
   <!-- Inclue gripper macro -->
   <xacro:include filename="$(find ariac_description)/urdf/vacuum_gripper/vacuum_gripper_macro.xacro"/>
-  <xacro:arg name="initial_positions_file" default="$(find ariac_description)/config/floor_robot_initial_positions.yaml"/>
+  <xacro:arg name="initial_positions_file" default="$(find ariac_description)/config/ceiling_robot_initial_positions.yaml"/>
   <xacro:property name="initial_positions_file" default="$(arg initial_positions_file)"/>
   <!-- Create a world link -->
   <link name="world" />
-  <!-- Run linear actuator macro -->
-  <xacro:linear_actuator
+  <!-- Run gantry macro -->
+  <xacro:gantry
     parent="world"
+    long_rail_length="15.0"
+    long_rail_width="0.2"
+    long_rail_offset="-5.0"
+    small_rail_length="15.0"
+    small_rail_width="0.2"
+    rail_height="2.9"
+    rail_thickness="0.1"
+    torso_height="-2.3"
     initial_positions="${load_yaml(initial_positions_file)}"
     >
-  </xacro:linear_actuator>
+  </xacro:gantry>
   <!-- Run ur macro -->
   <xacro:ur_robot
-    name="floor_arm"
-    prefix="floor_"
-    parent="robot_base"
+    name="ceiling_arm"
+    prefix="ceiling_"
+    parent="torso_main"
     joint_limits_parameters_file="$(find ur_description)/config/ur10e/joint_limits.yaml"
     kinematics_parameters_file="$(find ur_description)/config/ur10e/default_kinematics.yaml"
@@ -28,10 +36,10 @@
     sim_gazebo="true"
     initial_positions="${load_yaml(initial_positions_file)}">
-    <origin xyz="0 0 0.025" rpy="0 0 0" />
+    <origin xyz="0.51 0.0 1.3" rpy="0 1.57 0" />
   </xacro:ur_robot>
   <!-- Run gripper macro -->
   <xacro:vacuum_gripper
     parent="wrist_3_link"
-    prefix="floor"
+    prefix="ceiling"
     >
   </xacro:vacuum_gripper>
@@ -39,12 +47,12 @@
     reference="world">
   </gazebo>
-  <xacro:arg name="controllers" default="$(find ariac_description)/config/floor_robot_controllers.yaml" />
+  <xacro:arg name="controllers" default="$(find ariac_description)/config/ceiling_robot_controllers.yaml" />
   <gazebo>
     <plugin filename="libgazebo_ros2_control.so" name="gazebo_ros2_control">
       <ros>
-        <namespace>/floor</namespace>
+        <namespace>/ceiling</namespace>
       </ros>
       <parameters>$(arg controllers)</parameters>
-      <robot_param_node>/floor/robot_state_publisher</robot_param_node>
+      <robot_param_node>/ceiling/robot_state_publisher</robot_param_node>
     </plugin>
   </gazebo>

File: ariac_description/urdf/ceiling_robot/gantry_macro.xacro (robot description, xacro)
@@ -13,5 +13,5 @@
     initial_positions">
     <!-- ROS2 Control -->
-    <xacro:include filename="$(find ariac_description)/urdf/gantry.ros2_control.xacro"/>
+    <xacro:include filename="$(find ariac_description)/urdf/ceiling_robot/gantry.ros2_control.xacro"/>
     <xacro:gantry_ros2_control
       name="gantry"

File: ariac_description/urdf/floor_robot/floor_robot.urdf.xacro (robot description, xacro)
@@ -1,33 +1,25 @@
 <?xml version="1.0" ?>
-<robot name="ceiling_robot" xmlns:xacro="http://ros.org/wiki/xacro">
-  <!-- Include gantry macro -->
-  <xacro:include filename="$(find ariac_description)/urdf/gantry_macro.xacro"/>
+<robot name="floor_robot" xmlns:xacro="http://ros.org/wiki/xacro">
+  <!-- Include linear actuator macro -->
+  <xacro:include filename="$(find ariac_description)/urdf/floor_robot/linear_actuator_macro.xacro"/>
   <!-- Inclue ur robot macro -->
   <xacro:include filename="$(find ur_description)/urdf/ur_macro.xacro"/>
   <!-- Inclue gripper macro -->
   <xacro:include filename="$(find ariac_description)/urdf/vacuum_gripper/vacuum_gripper_macro.xacro"/>
-  <xacro:arg name="initial_positions_file" default="$(find ariac_description)/config/ceiling_robot_initial_positions.yaml"/>
+  <xacro:arg name="initial_positions_file" default="$(find ariac_description)/config/floor_robot_initial_positions.yaml"/>
   <xacro:property name="initial_positions_file" default="$(arg initial_positions_file)"/>
   <!-- Create a world link -->
   <link name="world" />
-  <!-- Run gantry macro -->
-  <xacro:gantry
+  <!-- Run linear actuator macro -->
+  <xacro:linear_actuator
     parent="world"
-    long_rail_length="15.0"
-    long_rail_width="0.2"
-    long_rail_offset="-5.0"
-    small_rail_length="15.0"
-    small_rail_width="0.2"
-    rail_height="2.9"
-    rail_thickness="0.1"
-    torso_height="-2.3"
     initial_positions="${load_yaml(initial_positions_file)}"
     >
-  </xacro:gantry>
+  </xacro:linear_actuator>
   <!-- Run ur macro -->
   <xacro:ur_robot
-    name="ceiling_arm"
-    prefix="ceiling_"
-    parent="torso_main"
+    name="floor_arm"
+    prefix="floor_"
+    parent="robot_base"
     joint_limits_parameters_file="$(find ur_description)/config/ur10e/joint_limits.yaml"
     kinematics_parameters_file="$(find ur_description)/config/ur10e/default_kinematics.yaml"
@@ -36,10 +28,10 @@
     sim_gazebo="true"
     initial_positions="${load_yaml(initial_positions_file)}">
-    <origin xyz="0.51 0.0 1.3" rpy="0 1.57 0" />
+    <origin xyz="0 0 0.025" rpy="0 0 0" />
   </xacro:ur_robot>
   <!-- Run gripper macro -->
   <xacro:vacuum_gripper
     parent="wrist_3_link"
-    prefix="ceiling"
+    prefix="floor"
     >
   </xacro:vacuum_gripper>
@@ -47,12 +39,12 @@
     reference="world">
   </gazebo>
-  <xacro:arg name="controllers" default="$(find ariac_description)/config/ceiling_robot_controllers.yaml" />
+  <xacro:arg name="controllers" default="$(find ariac_description)/config/floor_robot_controllers.yaml" />
   <gazebo>
     <plugin filename="libgazebo_ros2_control.so" name="gazebo_ros2_control">
       <ros>
-        <namespace>/ceiling</namespace>
+        <namespace>/floor</namespace>
       </ros>
       <parameters>$(arg controllers)</parameters>
-      <robot_param_node>/ceiling/robot_state_publisher</robot_param_node>
+      <robot_param_node>/floor/robot_state_publisher</robot_param_node>
     </plugin>
   </gazebo>

File: ariac_description/urdf/floor_robot/linear_actuator_macro.xacro (robot description, xacro)
@@ -5,5 +5,5 @@
     initial_positions">
     <!-- ROS2 Control -->
-    <xacro:include filename="$(find ariac_description)/urdf/linear_actuator.ros2_control.xacro"/>
+    <xacro:include filename="$(find ariac_description)/urdf/floor_robot/linear_actuator.ros2_control.xacro"/>
     <xacro:gantry_ros2_control
       name="linear_actuator"
