Commit message: fixed MoveIt issues and updated ReadMe

File: ariac_description/urdf/floor_robot/linear_actuator_macro.xacro (robot description, xacro)
@@ -17,9 +17,9 @@
         <origin xyz="0 0 0"/>
       </visual>
-      <collision>
+      <!-- <collision>
         <geometry>
           <box size="0.2 10 0.1"/>
         </geometry>
-      </collision>
+      </collision> -->
       <inertial>
         <mass value="100"/>
