Commit message: improved moveit configuration and test_competitor pick part demo

File: ariac_description/urdf/floor_robot/floor_robot.urdf.xacro (robot description, xacro)
@@ -28,5 +28,5 @@
     sim_gazebo="true"
     initial_positions="${load_yaml(initial_positions_file)}">
-    <origin xyz="0 0 0.025" rpy="0 0 0" />
+    <origin xyz="0 0 0.06" rpy="0 0 0" />
   </xacro:ur_robot>
   <!-- Run gripper macro -->

File: ariac_description/urdf/floor_robot/linear_actuator_macro.xacro (robot description, xacro)
@@ -17,9 +17,9 @@
         <origin xyz="0 0 0"/>
       </visual>
-      <!-- <collision>
+      <collision>
         <geometry>
           <box size="0.2 10 0.1"/>
         </geometry>
-      </collision> -->
+      </collision>
       <inertial>
         <mass value="100"/>

File: ariac_description/urdf/vacuum_gripper/vacuum_gripper_macro.xacro (robot description, xacro)
@@ -31,5 +31,5 @@
       <parent link="${prefix}_${parent}"/>
       <child link="${prefix}_gripper"/>
-      <limit lower="0" upper="0" effort="0" velocity="0" />
+      <limit lower="-.1" upper=".1" effort="0" velocity="0" />
       <origin xyz="0.0 0.0 0.01" rpy="0.0 0.0 0.0"/>
     </joint>
@@ -57,4 +57,14 @@
       </plugin>
     </gazebo>
+    <ros2_control name="${prefix}_gripper_control" type="system">
+      <hardware>
+        <plugin>gazebo_ros2_control/GazeboSystem</plugin>
+      </hardware>
+      <joint name="${prefix}_gripper_joint">
+        <state_interface name="position">
+          <param name="initial_value">0</param>
+        </state_interface>
+      </joint>
+    </ros2_control>
   </xacro:macro>
 </robot>

Commit message: fixed normal calculation

File: ariac_description/urdf/floor_robot/floor_robot.urdf.xacro (robot description, xacro)
@@ -28,5 +28,5 @@
     sim_gazebo="true"
     initial_positions="${load_yaml(initial_positions_file)}">
-    <origin xyz="0 0 0.06" rpy="0 0 0" />
+    <origin xyz="0 0 0.05" rpy="0 0 0" />
   </xacro:ur_robot>
   <!-- Run gripper macro -->
