Commit message: added agvs to ariac_robots description and reworked controller names also removed custom_ros2_control

File: ariac_description/urdf/ariac_robots/ariac_robots.urdf.xacro (robot description, xacro)
@@ -3,10 +3,36 @@
   <!-- Root link -->
   <link name="world"/>
+  <!-- Material for RVIZ -->
+  <material name="Grey">
+    <color rgba="${220/255} ${220/255} ${220/255} 1.0"/>
+  </material>
+  <!-- Locate Robot Macros -->
   <xacro:include filename="$(find ariac_description)/urdf/floor_robot/floor_robot_macro.xacro"/>
   <xacro:include filename="$(find ariac_description)/urdf/ceiling_robot/ceiling_robot_macro.xacro"/>
+  <xacro:include filename="$(find ariac_description)/urdf/agv/agv_macro.xacro"/>
   <!-- Floor Robot -->
   <xacro:floor_robot/>
   <!-- Ceiling Robot -->
   <xacro:ceiling_robot/>
+  <!-- AGV1 -->
+  <xacro:agv
+    agv_number="agv1"
+    y_position="4.8" >
+  </xacro:agv>
+  <!-- AGV2 -->
+  <xacro:agv
+    agv_number="agv2"
+    y_position="1.2" >
+  </xacro:agv>
+  <!-- AGV3 -->
+  <xacro:agv
+    agv_number="agv3"
+    y_position="-1.2" >
+  </xacro:agv>
+  <!-- AGV4 -->
+  <xacro:agv
+    agv_number="agv4"
+    y_position="-4.8" >
+  </xacro:agv>
   <gazebo
     reference="world">
@@ -19,5 +45,4 @@
       </ros>
       <parameters>$(arg controllers)</parameters>
-      <controller_manager_prefix>ariac_robots</controller_manager_prefix>
     </plugin>
   </gazebo>

File: ariac_description/urdf/ceiling_robot/gantry.ros2_control.xacro (robot description, xacro)
@@ -8,5 +8,5 @@
         <plugin>gazebo_ros2_control/GazeboSystem</plugin>
       </hardware>
-      <joint name="small_long_joint">
+      <joint name="gantry_x_axis_joint">
         <command_interface name="position">
           <param name="min">-12.4</param>
@@ -23,5 +23,5 @@
         <state_interface name="effort"/>
       </joint>
-      <joint name="torso_rail_joint">
+      <joint name="gantry_y_axis_joint">
         <command_interface name="position">
           <param name="min">-7</param>
@@ -38,5 +38,5 @@
         <state_interface name="effort"/>
       </joint>
-      <joint name="torso_base_main_joint">
+      <joint name="gantry_rotation_joint">
         <command_interface name="position">
           <param name="min">{-2*pi}</param>
@@ -53,5 +53,5 @@
         <state_interface name="effort"/>
       </joint>
-      <joint name="torso_main_torso_tray_joint">
+      <joint name="gantry_tray_joint">
         <state_interface name="position">
           <param name="initial_value">0</param>

File: ariac_description/urdf/ceiling_robot/gantry_macro.xacro (robot description, xacro)
@@ -31,4 +31,5 @@
           <box size="${long_rail_width} ${long_rail_length} ${rail_thickness}"/>
         </geometry>
+        <material name="Grey"/>
       </visual>
       <inertial>
@@ -62,4 +63,5 @@
           <box size="${long_rail_width} ${long_rail_length} ${rail_thickness}"/>
         </geometry>
+        <material name="Grey"/>
       </visual>
       <inertial>
@@ -92,4 +94,5 @@
           <box size="${small_rail_width} ${small_rail_length} ${rail_thickness}"/>
         </geometry>
+        <material name="Grey"/>
       </visual>
       <inertial>
@@ -105,5 +108,5 @@
       <material>Gazebo/GreyTransparent</material>
     </gazebo>
-    <joint name="small_long_joint" type="prismatic">
+    <joint name="gantry_x_axis_joint" type="prismatic">
       <parent link="long_rail_2"/>
       <child link="small_rail"/>
@@ -139,5 +142,5 @@
       <selfCollide>1</selfCollide>
     </gazebo>
-    <joint name="torso_rail_joint" type="prismatic">
+    <joint name="gantry_y_axis_joint" type="prismatic">
       <parent link="small_rail"/>
       <child link="torso_base"/>
@@ -181,5 +184,5 @@
       <selfCollide>1</selfCollide>
     </gazebo>
-    <joint name="torso_base_main_joint" type="revolute">
+    <joint name="gantry_rotation_joint" type="revolute">
       <parent link="torso_base"/>
       <child link="torso_main"/>
@@ -215,5 +218,5 @@
     <!-- We have to make this a non-fixed joint otherwise it is not recofnized by Gazebo -->
     <!-- The limit will not allow the joint to move -->
-    <joint name="torso_main_torso_tray_joint" type="revolute">
+    <joint name="gantry_tray_joint" type="revolute">
       <parent link="torso_main"/>
       <child link="torso_tray"/>

File: ariac_description/urdf/floor_robot/linear_actuator.ros2_control.xacro (robot description, xacro)
@@ -8,5 +8,5 @@
         <plugin>gazebo_ros2_control/GazeboSystem</plugin>
       </hardware>
-      <joint name="linear_actuator">
+      <joint name="linear_actuator_joint">
       <command_interface name="position">
         <param name="min">-4.8</param>

File: ariac_description/urdf/floor_robot/linear_actuator_macro.xacro (robot description, xacro)
@@ -16,4 +16,5 @@
         </geometry>
         <origin xyz="0 0 0"/>
+        <material name="Grey"/>
       </visual>
       <collision>
@@ -41,5 +42,5 @@
       <origin xyz="-1.3 0.0 0.93" rpy="0.0 0.0 ${pi}"/>
     </joint>
-    <joint name="linear_actuator" type="prismatic">
+    <joint name="linear_actuator_joint" type="prismatic">
       <axis xyz="0 1 0"/>
       <origin xyz="0.0 0.0 0.0"/>

File: ariac_description/urdf/vacuum_gripper/vacuum_gripper_macro.xacro (robot description, xacro)
@@ -10,4 +10,5 @@
           <mesh filename="file://$(find ariac_description)/meshes/vacuum_gripper/vacuum_gripper.stl" scale="1 1 1"/>
         </geometry>
+        <material name="Grey"/>
       </visual>
       <collision name="${prefix}_gripper_collision">
@@ -55,5 +56,4 @@
       <plugin filename="libVacuumGripperPlugin.so" name="${prefix}_vacuum_gripper_plugin">
         <ros>
-          <namespace>${prefix}_robot</namespace>
         </ros>
         <gripper_link>${prefix}_gripper</gripper_link>
