Commit message: setup vacuum gripper to detect contacts

File: ariac_description/urdf/vacuum_gripper/vacuum_gripper_macro.xacro (robot description, xacro)
@@ -6,11 +6,14 @@
     <link name="${prefix}_gripper">
       <visual>
+        <origin xyz="0 0 0" rpy="0 0 0"/>
         <geometry>
           <mesh filename="file://$(find ariac_description)/meshes/vacuum_gripper/vacuum_gripper.stl" scale="1 1 1"/>
         </geometry>
       </visual>
-      <collision>
+      <collision name="${prefix}_gripper_collision">
+        <origin xyz="0 0 -0.005" rpy="0 0 0"/>
         <geometry>
-          <mesh filename="file://$(find ariac_description)/meshes/vacuum_gripper/vacuum_gripper.stl" scale="1 1 1"/>
+          <!-- <mesh filename="file://$(find ariac_description)/meshes/vacuum_gripper/vacuum_gripper.stl" scale="1 1 1"/> -->
+          <cylinder radius="0.05" length="0.01" />
         </geometry>
       </collision>
@@ -24,21 +27,34 @@
       <material>Gazebo/Black</material>
     </gazebo>
-    <joint name="${prefix}_robot_to_gripper" type="fixed">
+    <joint name="${prefix}_gripper_joint" type="revolute">
+      <axis xyz="0 0 1"/>
       <parent link="${prefix}_${parent}"/>
       <child link="${prefix}_gripper"/>
+      <limit lower="0" upper="0" effort="0" velocity="0" />
       <origin xyz="0.0 0.0 0.01" rpy="0.0 0.0 0.0"/>
     </joint>
-    <!-- <gazebo>
-      <plugin name='vacuum_gripper' filename='libgazebo_ros_vacuum_gripper.so'>
+    <!-- Add a contact sensor to the gripper -->
+    <gazebo reference="${prefix}_gripper">
+      <sensor type="contact" name="bumper">
+        <update_rate>10</update_rate>
+        <contact>
+          <collision>${prefix}_gripper_collision_collision</collision>
+        </contact>
+        <plugin name="${prefix}_gripper_contact_sensor" filename="libgazebo_ros_bumper.so">
+          <ros>
+            <namespace>${prefix}_robot</namespace>
+          </ros>
+          <frame_name>${prefix}_gripper</frame_name>
+        </plugin>
+      </sensor>
+    </gazebo>
+    <gazebo>
+      <plugin filename="libvacuum_gripper.so" name="${prefix}_vacuum_gripper_plugin">
         <ros>
-          <namespace>/${prefix}</namespace>
-          <remapping>switch:=activate_gripper</remapping>
-          <remapping>grasping:=gripper_state</remapping>
+          <namespace>${prefix}_robot</namespace>
         </ros>
-        <link_name>${prefix}_gripper</link_name>
-        <max_distance>10.0</max_distance>
-        <fixed>ground_plane</fixed>
+        <gripper_link>${prefix}_gripper</gripper_link>
       </plugin>
-    </gazebo> -->
+    </gazebo>
   </xacro:macro>
 </robot>

Commit message: added service to change gripper color

File: ariac_description/urdf/vacuum_gripper/vacuum_gripper_macro.xacro (robot description, xacro)
@@ -5,5 +5,5 @@
     prefix">
     <link name="${prefix}_gripper">
-      <visual>
+      <visual name="${prefix}_gripper_visual">
         <origin xyz="0 0 0" rpy="0 0 0"/>
         <geometry>
@@ -24,4 +24,17 @@
       </inertial>
     </link>
+    <gazebo reference="${prefix}_gripper">
+      <visual name="${prefix}_gripper_visual">
+        <origin xyz="0 0 0" rpy="0 0 0"/>
+        <geometry>
+          <!-- <mesh filename="file://$(find ariac_description)/meshes/vacuum_gripper/vacuum_gripper.stl" scale="1 1 1"/> -->
+        </geometry>
+        <plugin filename="libgripper_change_plugin.so" name="${prefix}_gripper_change_plugin">
+          <ros>
+          </ros>
+          <robot_name>${prefix}_robot</robot_name>
+        </plugin>
+      </visual>
+    </gazebo>
     <gazebo reference="${prefix}_gripper">
       <material>Gazebo/Black</material>

Commit message: created new service to allow for changing between a tray gripper and a part gripper

File: ariac_description/urdf/vacuum_gripper/vacuum_gripper_macro.xacro (robot description, xacro)
@@ -24,10 +24,7 @@
       </inertial>
     </link>
-    <!-- <gazebo reference="${prefix}_gripper">
+    <gazebo reference="${prefix}_gripper">
       <visual name="${prefix}_gripper_visual">
-        <origin xyz="0 0 0" rpy="0 0 0"/>
-        <geometry>
-        </geometry>
-        <plugin filename="libgripper_change_plugin.so" name="${prefix}_gripper_change_plugin">
+        <plugin filename="libGripperColorPlugin.so" name="${prefix}_gripper_color_plugin">
           <ros>
           </ros>
@@ -35,8 +32,8 @@
         </plugin>
       </visual>
+    </gazebo>
+    <!-- <gazebo reference="${prefix}_gripper">
+      <material>Gazebo/Black</material>
     </gazebo> -->
-    <gazebo reference="${prefix}_gripper">
-      <material>Gazebo/Black</material>
-    </gazebo>
     <joint name="${prefix}_gripper_joint" type="revolute">
       <axis xyz="0 0 1"/>
@@ -56,5 +53,5 @@
     </gazebo>
     <gazebo>
-      <plugin filename="libvacuum_gripper.so" name="${prefix}_vacuum_gripper_plugin">
+      <plugin filename="libVacuumGripperPlugin.so" name="${prefix}_vacuum_gripper_plugin">
         <ros>
           <namespace>${prefix}_robot</namespace>

Commit message: Incomplete work on task manager

File: ariac_description/urdf/vacuum_gripper/vacuum_gripper_macro.xacro (robot description, xacro)
@@ -10,4 +10,5 @@
           <mesh filename="file://$(find ariac_description)/meshes/vacuum_gripper/vacuum_gripper.stl" scale="1 1 1"/>
         </geometry>
+        <material name="Grey"/>
       </visual>
       <collision name="${prefix}_gripper_collision">
@@ -26,9 +27,5 @@
     <gazebo reference="${prefix}_gripper">
       <visual name="${prefix}_gripper_visual">
-        <origin xyz="0 0 0" rpy="0 0 0"/>
-        <geometry>
-          <!-- <mesh filename="file://$(find ariac_description)/meshes/vacuum_gripper/vacuum_gripper.stl" scale="1 1 1"/> -->
-        </geometry>
-        <plugin filename="libgripper_change_plugin.so" name="${prefix}_gripper_change_plugin">
+        <plugin filename="libGripperColorPlugin.so" name="${prefix}_gripper_color_plugin">
           <ros>
           </ros>
@@ -57,7 +54,6 @@
     </gazebo>
     <gazebo>
-      <plugin filename="libvacuum_gripper.so" name="${prefix}_vacuum_gripper_plugin">
+      <plugin filename="libVacuumGripperPlugin.so" name="${prefix}_vacuum_gripper_plugin">
         <ros>
-          <namespace>${prefix}_robot</namespace>
         </ros>
         <gripper_link>${prefix}_gripper</gripper_link>

Commit message: added functionality to complete a kitting task

File: ariac_description/urdf/vacuum_gripper/vacuum_gripper_macro.xacro (robot description, xacro)
@@ -41,5 +41,5 @@
       <parent link="${prefix}_${parent}"/>
       <child link="${prefix}_gripper"/>
-      <limit lower="-.1" upper=".1" effort="0" velocity="0" />
+      <limit lower="-.001" upper=".001" effort="1000" velocity="0" />
       <origin xyz="0.0 0.0 0.01" rpy="0.0 0.0 0.0"/>
     </joint>
